File: ESC_Control_Board_STM32G071.kicad_sch (KiCad schematic)
At the start: 6 parts, among them J1 Conn_01x02, J2 Conn_01x03, J3 Conn_01x04, J4 Conn_01x04, J5 Conn_01x02, J6 Conn_01x15

Commit message: Layout updates
Parts:
- removed J1: Conn_01x02, Connector_Molex:Molex_Micro-Fit_3.0_43650-0210_1x02-1MP_P3.00mm_Horizontal, symbol Connector_Generic:Conn_01x02
- J2: footprint Connector_Molex:Molex_Micro-Fit_3.0_43650-0310_1x03-1MP_P3.00mm_Horizontal -> MAG_Connectors:PWM_PADS
- J3, J4: footprint Connector_Molex:Molex_Micro-Fit_3.0_43650-0410_1x04-1MP_P3.00mm_Horizontal -> Connector_Molex:Molex_PicoBlade_53261-0471_1x04-1MP_P1.25mm_Horizontal
- J5: footprint Connector_Molex:Molex_Micro-Fit_3.0_43650-0210_1x02-1MP_P3.00mm_Horizontal -> Connector_Molex:Molex_PicoBlade_53261-0271_1x02-1MP_P1.25mm_Horizontal
Connections:
- net GND: now also J6.11 (Pin_11)
Other:
- sheet Power_Supplies ports: added none; removed VBATT
- note removed: "Battery"
