File: ESC_Control_Board_STM32G071.kicad_sch (KiCad schematic)
At the start: 5 parts, among them J2 Conn_01x03, J3 Conn_01x04, J4 Conn_01x04, J5 Conn_01x02, J6 Conn_01x15

Commit message: Updates for review
Other:
- added sheet Revision History (revision_history.kicad_sch)
- sheet CAN ports: added CAN1_CS, CAN2_CS, MISO, MOSI, SCK; removed CAN_RX1, CAN_RX2, CAN_TX1, CAN_TX2
- sheet MCU ports: added PB3, PB4, PB5, PB6; removed PB1, PC4, PC5, PD4, PD5
