File: PWM.kicad_sch (KiCad schematic)
At the start: 4 parts, among them IC5 ISO1540QDRQ1

Commit message: Layout updates
Parts:
- IC5: symbol MA_General:ISO1540QDRQ1 -> MAG_Isolators:ISO1540QDRQ1
Changed lines of the file:
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@@
     (pin "1")
   )
-  (symbol (lib_id "MA_General:ISO1540QDRQ1") (at 140.97 95.25 0) (unit 1)
+  (symbol (lib_id "MAG_Isolators:ISO1540QDRQ1") (at 140.97 95.25 0) (unit 1)
     (in_bom yes) (on_board yes) (fields_autoplaced)
     (property "Reference" "IC5" (id 0) (at 154.94 87.63 0))
