File: current_sense.kicad_sch (KiCad schematic)
At the start: 2 parts, among them IC6 INA240A2PW

Commit message: Layout updates
Parts:
- IC6: symbol MA_General:INA240A2PW -> MAG_Current_Sense_Amplifiers:INA240A2PW
Changed lines of the file:
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@@
     (pin "2")
   )
-  (symbol (lib_id "MA_General:INA240A2PW") (at 138.43 93.98 0) (unit 1)
+  (symbol (lib_id "MAG_Current_Sense_Amplifiers:INA240A2PW") (at 138.43 93.98 0) (unit 1)
     (in_bom yes) (on_board yes) (fields_autoplaced)
     (property "Reference" "IC6" (id 0) (at 152.4 86.36 0))
