File: power_supplies.kicad_sch (KiCad schematic)
At the start: 22 parts, among them IC4 AZ1117CR-3.3TRG1, U10 LNK306DN-TL

Commit message: Layout updates
Parts:
- removed C13: 100n, Capacitor_SMD:C_0603_1608Metric, symbol Device:C
- IC4: symbol MA_General:AZ1117CR-3.3TRG1 -> MAG_LDO_Regulators:AZ1117CR-3.3TRG1
- PS1: footprint AZ1117CR50TRG1 -> MAG_LDO_Regulators:AZ1117CR33TRG1; symbol MA_General:AZ1117CR-5.0TRG1 -> MAG_LDO_Regulators:AZ1117CR-5.0TRG1
- U10: footprint (none) -> MAG_Switching_Regulators:SOIC127P600X175-8N; symbol MA_General:LNK306DN-TL -> MAG_Switching_Regulators:LNK306DN-TL
Changed lines of the file:
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@@
   (junction (at 102.87 153.67) (diameter 0) (color 0 0 0 0)
   )
-  (junction (at 92.71 105.41) (diameter 0) (color 0 0 0 0)
-  )
   (junction (at 81.28 55.88) (diameter 0) (color 0 0 0 0)
   )
@@
     (stroke (width 0) (type default) (color 0 0 0 0))
   )
-  (wire (pts (xy 92.71 105.41) (xy 102.87 105.41))
+  (wire (pts (xy 86.36 105.41) (xy 102.87 105.41))
     (stroke (width 0) (type default) (color 0 0 0 0))
   )
@@
     (stroke (width 0) (type default) (color 0 0 0 0))
   )
-  (wire (pts (xy 86.36 105.41) (xy 92.71 105.41))
-    (stroke (width 0) (type default) (color 0 0 0 0))
-  )
   (wire (pts (xy 134.62 49.53) (xy 134.62 55.88))
     (stroke (width 0) (type default) (color 0 0 0 0))
@@
     (stroke (width 0) (type default) (color 0 0 0 0))
   )
-  (wire (pts (xy 92.71 105.41) (xy 92.71 109.22))
-    (stroke (width 0) (type default) (color 0 0 0 0))
-  )
   (wire (pts (xy 102.87 101.6) (xy 102.87 105.41))
     (stroke (width 0) (type default) (color 0 0 0 0))
@@
     (stroke (width 0) (type default) (color 0 0 0 0))
   )
-  (wire (pts (xy 92.71 116.84) (xy 92.71 120.65))
-    (stroke (width 0) (type default) (color 0 0 0 0))
-  )
   (wire (pts (xy 115.57 55.88) (xy 134.62 55.88))
     (stroke (width 0) (type default) (color 0 0 0 0))
@@
   (wire (pts (xy 50.8 44.45) (xy 50.8 45.72))
     (stroke (width 0) (type default) (color 0 0 0 0))
+  )
+  (global_label "VBATT" (shape input) (at 33.02 30.48 180) (fields_autoplaced)
+    (effects (font (size 1.27 1.27)) (justify right))
+    (property "Intersheet References" "${INTERSHEET_REFS}" (id 0) (at 25.2245 30.5594 0)
+      (effects (font (size 1.27 1.27)) (justify right) hide)
+    )
   )
   (hierarchical_label "VBATT_SENSE" (shape input) (at 59.69 45.72 0)
     (effects (font (size 1.27 1.27)) (justify left))
-  )
-  (hierarchical_label "VBATT" (shape input) (at 33.02 30.48 180)
-    (effects (font (size 1.27 1.27)) (justify right))
   )
   (symbol (lib_id "Device:C") (at 58.42 50.8 0) (unit 1)
@@
     (pin "2")
   )
-  (symbol (lib_id "Device:C") (at 92.71 113.03 0) (unit 1)
-    (in_bom yes) (on_board yes)
-    (property "Reference" "C13" (id 0) (at 95.25 111.76 0)
-      (effects (font (size 1.27 1.27)) (justify left))
-    )
-    (property "Value" "100n" (id 1) (at 95.25 114.3 0)
-      (effects (font (size 1.27 1.27)) (justify left))
-    )
-    (property "Footprint" "Capacitor_SMD:C_0603_1608Metric" (id 2) (at 93.6752 116.84 0)
-      (effects (font (size 1.27 1.27)) hide)
-    )
-    (property "Datasheet" "~" (id 3) (at 92.71 113.03 0)
-      (effects (font (size 1.27 1.27)) hide)
-    )
-    (pin "1")
-    (pin "2")
-  )
   (symbol (lib_id "power:GND") (at 58.42 71.12 0) (unit 1)
     (in_bom yes) (on_board yes) (fields_autoplaced)
@@
     (pin "1")
   )
-  (symbol (lib_id "MA_General:AZ1117CR-3.3TRG1") (at 54.61 152.4 0) (unit 1)
+  (symbol (lib_id "MAG_LDO_Regulators:AZ1117CR-3.3TRG1") (at 54.61 152.4 0) (unit 1)
     (in_bom yes) (on_board yes) (fields_autoplaced)
     (property "Reference" "IC4" (id 0) (at 71.12 144.78 0))
@@
     (pin "1")
   )
-  (symbol (lib_id "power:GND") (at 92.71 120.65 0) (unit 1)
-    (in_bom yes) (on_board yes) (fields_autoplaced)
-    (property "Reference" "#PWR0134" (id 0) (at 92.71 127 0)
-      (effects (font (size 1.27 1.27)) hide)
-    )
-    (property "Value" "GND" (id 1) (at 92.71 125.73 0))
-    (property "Footprint" "" (id 2) (at 92.71 120.65 0)
-      (effects (font (size 1.27 1.27)) hide)
-    )
-    (property "Datasheet" "" (id 3) (at 92.71 120.65 0)
-      (effects (font (size 1.27 1.27)) hide)
-    )
-    (pin "1")
-  )
   (symbol (lib_id "power:GND") (at 92.71 168.91 0) (unit 1)
     (in_bom yes) (on_board yes) (fields_autoplaced)
@@
     (pin "2")
   )
-  (symbol (lib_id "MA_General:AZ1117CR-5.0TRG1") (at 54.61 105.41 0) (unit 1)
+  (symbol (lib_id "MAG_LDO_Regulators:AZ1117CR-5.0TRG1") (at 54.61 105.41 0) (unit 1)
     (in_bom yes) (on_board yes) (fields_autoplaced)
     (property "Reference" "PS1" (id 0) (at 70.485 97.79 0))
     (property "Value" "AZ1117CR-5.0TRG1" (id 1) (at 70.485 100.33 0))
-    (property "Footprint" "AZ1117CR50TRG1" (id 2) (at 83.82 102.87 0)
+    (property "Footprint" "MAG_LDO_Regulators:AZ1117CR33TRG1" (id 2) (at 83.82 102.87 0)
       (effects (font (size 1.27 1.27)) (justify left) hide)
     )
@@
     (pin "4")
   )
-  (symbol (lib_id "MA_General:LNK306DN-TL") (at 66.04 35.56 0) (unit 1)
+  (symbol (lib_id "MAG_Switching_Regulators:LNK306DN-TL") (at 66.04 35.56 0) (unit 1)
     (in_bom yes) (on_board yes)
     (property "Reference" "U10" (id 0) (at 96.52 41.91 0))
     (property "Value" "LNK306DN-TL" (id 1) (at 96.52 44.45 0))
-    (property "Footprint" "" (id 2) (at 66.04 35.56 0)
-      (effects (font (size 1.27 1.27)) hide)
-    )
-    (property "Datasheet" "" (id 3) (at 66.04 35.56 0)
-      (effects (font (size 1.27 1.27)) hide)
-    )
-    (property "Reference_1" "IC" (id 4) (at 81.28 27.94 0)
-      (effects (font (size 1.27 1.27)) hide)
-    )
-    (property "Value_1" "LNK306DN-TL" (id 5) (at 81.28 30.48 0)
-      (effects (font (size 1.27 1.27)) hide)
+    (property "Footprint" "MAG_Switching_Regulators:SOIC127P600X175-8N" (id 2) (at 86.995 26.035 90)
+      (effects (font (size 1.27 1.27)) hide)
+    )
+    (property "Datasheet" "" (id 3) (at 86.995 26.035 90)
+      (effects (font (size 1.27 1.27)) hide)
+    )
+    (property "Reference_1" "IC" (id 4) (at 90.17 43.18 0)
+      (effects (font (size 1.27 1.27)) (justify left top))
+    )
+    (property "Value_1" "LNK306DN-TL" (id 5) (at 90.17 40.64 0)
+      (effects (font (size 1.27 1.27)) (justify left top))
     )
     (property "Footprint_1" "SOIC127P600X175-8N" (id 6) (at 92.71 130.48 0)
