File: untitled.kicad_sch (KiCad schematic)
At the start: 30 parts, among them U1 L6498DTR, U2 L6498DTR, U3 L6498DTR, U4 ZXGD3006E6QTA, U5 ZXGD3006E6QTA, U6 ZXGD3006E6QTA, U7 ZXGD3006E6QTA, U8 ZXGD3006E6QTA, U9 ZXGD3006E6QTA

Commit message: Layout updates
Parts:
- U1, U2, U3: footprint (none) -> MAG_Gate_Drivers:SOT127P600X175-8N; symbol MA_General:L6498DTR -> MAG_Gate_Drivers:L6498DTR
- U4, U5, U6, U7, U8, U9: footprint (none) -> MAG_Gate_Drivers:SOT95P285X140-6N; symbol MA_General:ZXGD3006E6QTA -> MAG_Gate_Drivers:ZXGD3006E6QTA
