File: MCU.kicad_sch (KiCad schematic)
At the start: 2 parts, among them IC3 STM32G071RBT6

Commit message: Layout updates
Parts:
- added J7: TC6NL_SWD, TC2030IDC, symbol MAG_Programming_Headers:TC6NL_SWD
- IC3: symbol MA_General:STM32G071RBT6 -> MAG_MCUs:STM32G071RBT6
Connections:
- net +3V3: now also J7.1
- net GND: now also J7.5
- net NRST: now reaches IC3.12 (PF2-NRST)
- net NRST: now also J7.3
- net SWO: now reaches IC3.20 (PA3)
- net SWO: now also J7.6
- net SWDIO: now reaches IC3.45 (PA13)
- net SWDIO: now also J7.2
- net SWCLK: now reaches IC3.46 (PA14-BOOT0)
- net SWCLK: now also J7.4
Other:
- note added: "Add oscillator!!"
- note added: "Add programming header"
Changed lines of the file:
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@@
   (junction (at 110.49 86.36) (diameter 0) (color 0 0 0 0)
   )
+  (wire (pts (xy 237.49 87.63) (xy 237.49 90.17))
+    (stroke (width 0) (type default) (color 0 0 0 0))
+  )
   (wire (pts (xy 147.32 127) (xy 147.32 146.05))
     (stroke (width 0) (type default) (color 0 0 0 0))
   )
+  (wire (pts (xy 238.76 87.63) (xy 237.49 87.63))
+    (stroke (width 0) (type default) (color 0 0 0 0))
+  )
   (wire (pts (xy 165.1 127) (xy 165.1 146.05))
     (stroke (width 0) (type default) (color 0 0 0 0))
@@
     (stroke (width 0) (type default) (color 0 0 0 0))
   )
+  (wire (pts (xy 237.49 80.01) (xy 237.49 82.55))
+    (stroke (width 0) (type default) (color 0 0 0 0))
+  )
+  (wire (pts (xy 144.78 127) (xy 144.78 146.05))
+    (stroke (width 0) (type default) (color 0 0 0 0))
+  )
   (wire (pts (xy 154.94 127) (xy 154.94 146.05))
     (stroke (width 0) (type default) (color 0 0 0 0))
   )
+  (wire (pts (xy 182.88 78.74) (xy 209.55 78.74))
+    (stroke (width 0) (type default) (color 0 0 0 0))
+  )
+  (wire (pts (xy 233.68 85.09) (xy 238.76 85.09))
+    (stroke (width 0) (type default) (color 0 0 0 0))
+  )
   (wire (pts (xy 144.78 44.45) (xy 144.78 58.42))
     (stroke (width 0) (type default) (color 0 0 0 0))
@@
     (stroke (width 0) (type default) (color 0 0 0 0))
   )
+  (wire (pts (xy 119.38 101.6) (xy 129.54 101.6))
+    (stroke (width 0) (type default) (color 0 0 0 0))
+  )
+  (wire (pts (xy 182.88 81.28) (xy 209.55 81.28))
+    (stroke (width 0) (type default) (color 0 0 0 0))
+  )
   (wire (pts (xy 137.16 127) (xy 137.16 146.05))
+    (stroke (width 0) (type default) (color 0 0 0 0))
+  )
+  (wire (pts (xy 259.08 82.55) (xy 265.43 82.55))
+    (stroke (width 0) (type default) (color 0 0 0 0))
+  )
+  (wire (pts (xy 259.08 87.63) (xy 265.43 87.63))
+    (stroke (width 0) (type default) (color 0 0 0 0))
+  )
+  (wire (pts (xy 237.49 82.55) (xy 238.76 82.55))
+    (stroke (width 0) (type default) (color 0 0 0 0))
+  )
+  (wire (pts (xy 259.08 85.09) (xy 265.43 85.09))
     (stroke (width 0) (type default) (color 0 0 0 0))
   )
@@
     (effects (font (size 1.27 1.27)) (justify left bottom))
   )
+  (text "Add oscillator!!" (at 229.87 54.61 0)
+    (effects (font (size 1.27 1.27)) (justify left bottom))
+  )
+  (text "Add programming header \n" (at 229.87 50.8 0)
+    (effects (font (size 1.27 1.27)) (justify left bottom))
+  )
   (text "Why duplicated?\n" (at 76.2 101.6 0)
     (effects (font (size 1.27 1.27)) (justify left bottom))
@@
     (effects (font (size 1.27 1.27)) (justify left bottom))
   )
+  (label "SWO" (at 265.43 87.63 180)
+    (effects (font (size 1.27 1.27)) (justify right bottom))
+  )
+  (label "SWDIO" (at 209.55 81.28 180)
+    (effects (font (size 1.27 1.27)) (justify right bottom))
+  )
   (label "VOLT_SENSE" (at 149.86 146.05 90)
     (effects (font (size 1.27 1.27)) (justify left bottom))
@@
     (effects (font (size 1.27 1.27)) (justify right bottom))
   )
+  (label "SWO" (at 144.78 146.05 90)
+    (effects (font (size 1.27 1.27)) (justify left bottom))
+  )
   (label "USART2_TX" (at 160.02 54.61 90)
     (effects (font (size 1.27 1.27)) (justify left bottom))
@@
     (effects (font (size 1.27 1.27)) (justify left bottom))
   )
+  (label "NRST" (at 233.68 85.09 0)
+    (effects (font (size 1.27 1.27)) (justify left bottom))
+  )
   (label "pV_HIGH" (at 208.28 86.36 180)
     (effects (font (size 1.27 1.27)) (justify right bottom))
   )
+  (label "NRST" (at 119.38 101.6 0)
+    (effects (font (size 1.27 1.27)) (justify left bottom))
+  )
   (label "pW_COMP" (at 137.16 146.05 90)
     (effects (font (size 1.27 1.27)) (justify left bottom))
@@
     (effects (font (size 1.27 1.27)) (justify right bottom))
   )
+  (label "SWDIO" (at 265.43 82.55 180)
+    (effects (font (size 1.27 1.27)) (justify right bottom))
+  )
   (label "pW_HIGH" (at 208.28 104.14 180)
     (effects (font (size 1.27 1.27)) (justify right bottom))
   )
+  (label "SWCLK" (at 209.55 78.74 180)
+    (effects (font (size 1.27 1.27)) (justify right bottom))
+  )
   (label "CAN2_EN" (at 162.56 53.34 90)
     (effects (font (size 1.27 1.27)) (justify left bottom))
@@
   (label "CAN1_EN" (at 165.1 146.05 90)
     (effects (font (size 1.27 1.27)) (justify left bottom))
+  )
+  (label "SWCLK" (at 265.43 85.09 180)
+    (effects (font (size 1.27 1.27)) (justify right bottom))
   )
   (hierarchical_label "PD6" (shape input) (at 157.48 44.45 90)
@@
     (pin "2")
   )
+  (symbol (lib_id "MAG_Programming_Headers:TC6NL_SWD") (at 238.76 82.55 0) (unit 1)
+    (in_bom yes) (on_board yes) (fields_autoplaced)
+    (property "Reference" "J7" (id 0) (at 248.92 74.93 0))
+    (property "Value" "TC6NL_SWD" (id 1) (at 248.92 77.47 0))
+    (property "Footprint" "TC2030IDC" (id 2) (at 255.27 80.01 0)
+      (effects (font (size 1.27 1.27)) (justify left) hide)
+    )
+    (property "Datasheet" "https://datasheet.datasheetarchive.com/originals/distributors/Datasheets_SAMA/62bc384e093448baaaa63dbd0b9d8707.pdf" (id 3) (at 255.27 82.55 0)
+      (effects (font (size 1.27 1.27)) (justify left) hide)
+    )
+    (property "Description" "CABLE ADAPTER 6 POS" (id 4) (at 255.27 85.09 0)
+      (effects (font (size 1.27 1.27)) (justify left) hide)
+    )
+    (property "Height" "19" (id 5) (at 255.27 87.63 0)
+      (effects (font (size 1.27 1.27)) (justify left) hide)
+    )
+    (property "Manufacturer_Name" "Tag Connect" (id 6) (at 255.27 90.17 0)
+      (effects (font (size 1.27 1.27)) (justify left) hide)
+    )
+    (property "Manufacturer_Part_Number" "TC2030-IDC" (id 7) (at 255.27 92.71 0)
+      (effects (font (size 1.27 1.27)) (justify left) hide)
+    )
+    (property "Mouser Part Number" "" (id 8) (at 255.27 95.25 0)
+      (effects (font (size 1.27 1.27)) (justify left) hide)
+    )
+    (property "Mouser Price/Stock" "" (id 9) (at 255.27 97.79 0)
+      (effects (font (size 1.27 1.27)) (justify left) hide)
+    )
+    (property "Arrow Part Number" "" (id 10) (at 255.27 100.33 0)
+      (effects (font (size 1.27 1.27)) (justify left) hide)
+    )
+    (property "Arrow Price/Stock" "" (id 11) (at 255.27 102.87 0)
+      (effects (font (size 1.27 1.27)) (justify left) hide)
+    )
+    (property "Mouser Testing Part Number" "" (id 12) (at 255.27 105.41 0)
+      (effects (font (size 1.27 1.27)) (justify left) hide)
+    )
+    (property "Mouser Testing Price/Stock" "" (id 13) (at 255.27 107.95 0)
+      (effects (font (size 1.27 1.27)) (justify left) hide)
+    )
+    (pin "1")
+    (pin "2")
+    (pin "3")
+    (pin "4")
+    (pin "5")
+    (pin "6")
+  )
   (symbol (lib_id "power:+3V3") (at 110.49 86.36 0) (unit 1)
     (in_bom yes) (on_board yes) (fields_autoplaced)
@@
     (pin "1")
   )
+  (symbol (lib_id "power:GND") (at 237.49 90.17 0) (unit 1)
+    (in_bom yes) (on_board yes) (fields_autoplaced)
+    (property "Reference" "#PWR02" (id 0) (at 237.49 96.52 0)
+      (effects (font (size 1.27 1.27)) hide)
+    )
+    (property "Value" "GND" (id 1) (at 237.49 95.25 0))
+    (property "Footprint" "" (id 2) (at 237.49 90.17 0)
+      (effects (font (size 1.27 1.27)) hide)
+    )
+    (property "Datasheet" "" (id 3) (at 237.49 90.17 0)
+      (effects (font (size 1.27 1.27)) hide)
+    )
+    (pin "1")
+  )
+  (symbol (lib_id "power:+3V3") (at 237.49 80.01 0) (unit 1)
+    (in_bom yes) (on_board yes) (fields_autoplaced)
+    (property "Reference" "#PWR01" (id 0) (at 237.49 83.82 0)
+      (effects (font (size 1.27 1.27)) hide)
+    )
+    (property "Value" "+3V3" (id 1) (at 237.49 74.93 0))
+    (property "Footprint" "" (id 2) (at 237.49 80.01 0)
+      (effects (font (size 1.27 1.27)) hide)
+    )
+    (property "Datasheet" "" (id 3) (at 237.49 80.01 0)
+      (effects (font (size 1.27 1.27)) hide)
+    )
+    (pin "1")
+  )
   (symbol (lib_id "power:GND") (at 110.49 95.25 0) (unit 1)
     (in_bom yes) (on_board yes) (fields_autoplaced)
@@
     (pin "1")
   )
-  (symbol (lib_id "MA_General:STM32G071RBT6") (at 129.54 73.66 0) (unit 1)
+  (symbol (lib_id "MAG_MCUs:STM32G071RBT6") (at 129.54 73.66 0) (unit 1)
     (in_bom yes) (on_board yes) (fields_autoplaced)
     (property "Reference" "IC3" (id 0) (at 186.69 67.0812 0))

Commit message: Updates for review
Parts:
- removed J7: TC6NL_SWD, TC2030IDC, symbol MAG_Programming_Headers:TC6NL_SWD
- added J1: Conn_ARM_JTAG_SWD_10, Connector:Tag-Connect_TC2050-IDC-NL_2x05_P1.27mm_Vertical_with_bottom_clip, symbol Connector:Conn_ARM_JTAG_SWD_10
Connections:
- net +3V3: now also J1.1 (VTref)
- net GND: now also J1.3 (GND), J1.5 (GND), J1.9 (GNDDetect)
- net NRST: now also J1.10 (~{RESET})
- net SWCLK: now also J1.4 (SWDCLK/TCK)
- net SWDIO: now also J1.2 (SWDIO/TMS)
- net SWO: now also J1.6 (SWO/TDO)
- net PC0: now reaches IC3.13 (PC0)
- net PC1: now reaches IC3.14 (PC1)
- net PC2: now reaches IC3.15 (PC2)
- net TDI: now reaches IC3.47 (PA15)
- net TDI: now also J1.8 (NC/TDI)
- net PB3: now reaches IC3.57 (PB3)
- net PB4: now reaches IC3.58 (PB4)
- net PB5: now reaches IC3.59 (PB5)
- net PB6: now reaches IC3.60 (PB6)
- net PC4: no longer names the net of IC3.25 (PC4)
- net PC5: no longer names the net of IC3.26 (PC5)
- net PD4: no longer names the net of IC3.54 (PD4)
- net PD5: no longer names the net of IC3.55 (PD5)
- no-connect marks 0 -> 36
Other:
- note removed: "Add oscillator!!"
- note removed: "Add programming header"
