File: hw/current_sense.kicad_sch (KiCad schematic)
At the start: 2 parts, among them IC6 INA240A2PW

Commit message: Revision V1.0
Other:
- note added: "Only good for 80V CMR"
- note added: "Replace with isolated Si8920!"
Changed lines of the file:
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@@
+    (effects (font (size 1.27 1.27)) (justify left bottom))
+  )
+  (text "Replace with isolated Si8920!\n" (at 139.7 72.39 0)
+    (effects (font (size 1.27 1.27)) (justify left bottom))
+  )
+  (text "Only good for 80V CMR\n\n" (at 140.97 119.38 0)
     (effects (font (size 1.27 1.27)) (justify left bottom))
   )

Commit message: update comments
Parts:
- C25: Manufacturer_Name (none) -> Murata; Manufacturer_Part_Number (none) -> GRT188C81E475KE13D
Changed lines of the file:
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@@
+      (effects (font (size 1.27 1.27)) hide)
+    )
+    (property "Manufacturer_Name" "Murata" (id 4) (at 177.8 97.79 0)
+      (effects (font (size 1.27 1.27)) hide)
+    )
+    (property "Manufacturer_Part_Number" "GRT188C81E475KE13D " (id 5) (at 177.8 97.79 0)
       (effects (font (size 1.27 1.27)) hide)
     )
