File: hw/ESC_Control_Board_STM32G071_V2.kicad_pcb (KiCad board)
At the start: 6 copper layers, 50 x 67 mm, 90 parts, among them IC1 MCP2518FDT-E_SL, IC2 MCP2518FDT-E_SL, IC3 STM32G071RBT6, IC4 AZ1117CR-3.3TRG1, IC5 ISO1540QDRQ1, IC6 INA240A2PW, IC7 ADM3050EBRIZ, IC8 ADM3050EBRIZ, J1 Conn_ARM_JTAG_SWD_10, J2 Conn_01x03, J3 Conn_01x04, J4 Conn_01x04, J5 Conn_01x02, J6 Conn_01x15, U1 L6498DTR, U10 LNK306DN-TL, U2 L6498DTR, U3 L6498DTR, U4 ZXGD3006E6QTA, U5 ZXGD3006E6QTA, U6 ZXGD3006E6QTA, U7 ZXGD3006E6QTA, U8 ZXGD3006E6QTA, U9 ZXGD3006E6QTA, Y1 ABM8-20.000MHZ-10-B1U-T, Y2 ABM8-20.000MHZ-10-B1U-T

Commit message: commenting
Parts:
- removed C1, C2, C25, C29, C3, C30, C4, C9: 4u7, Capacitor_SMD:C_0603_1608Metric
- removed C13, C26, C27, C28: 12p, Capacitor_SMD:C_0603_1608Metric
- removed C15: 47u, Capacitor_SMD:C_1210_3225Metric
- removed IC1, IC2: MCP2518FDT-E_SL, MAG_CAN_Transceivers:SOIC127P600X175-14N
- removed IC3: STM32G071RBT6, MAG_ESC:QFP50P1200X1200X160-64N
- removed IC6: INA240A2PW, MAG_Current_Sense_Amplifiers:SOP65P640X120-8N
- removed IC7, IC8: ADM3050EBRIZ, MAG_CAN_Transceivers:SOIC127P1031X265-8N
- removed J4: Conn_01x04, Connector_Molex:Molex_PicoBlade_53261-0471_1x04-1MP_P1.25mm_Horizontal
- removed J5: Conn_01x02, Connector_Molex:Molex_PicoBlade_53261-0271_1x02-1MP_P1.25mm_Horizontal
- removed PS1: AZ1117CR-5.0TRG1, MAG_LDO_Regulators:AZ1117CR33TRG1
- removed Y1, Y2: ABM8-20.000MHZ-10-B1U-T, MAG_Crystals:ABM810000MHZ12D2W
- added U11: STM32G071GBU6, MAG_MCUs:UFQFPN-28, F.Cu at (127.3, 55.3)
- J3: value Conn_01x04 -> Conn_01x01_Pin; footprint Connector_Molex:Molex_PicoBlade_53261-0471_1x04-1MP_P1.25mm_Horizontal -> TestPoint:TestPoint_Pad_1.0x1.0mm
- U10: footprint MAG_Switching_Regulators:SOIC127P600X175-8N -> MAG_Switching_Regulators:SOIC127P600X175-8N_MISSING_PIN
- moved J3 48.2 mm to (125.6, 60.4), turned to 0 degrees
- moved C23 6.26 mm to (118.3, 50.2), turned to 180 degrees
- moved R22 5.06 mm to (118.3, 51.7), turned to 180 degrees
- moved R14 4.54 mm to (117.5, 58.1), turned to 180 degrees
- moved R20 4.22 mm to (117.5, 54.9), turned to 180 degrees
- moved C5 3.20 mm to (123.0, 54.9)
- moved C12 2.74 mm to (117.5, 56.6), turned to 180 degrees
- moved C22 2.42 mm to (117.5, 53.4), turned to 180 degrees
- moved C21 1.55 mm to (117.5, 60.4), turned to 180 degrees
- moved R18 1.15 mm to (117.5, 61.9), turned to 180 degrees
- moved U4 0.34 mm to (147.6, 75.9)
- moved R13 0.15 mm to (152.8, 76.0)
- moved C6 0.13 mm to (146.2, 71.9)
- turned R23 to 90 degrees
Connections:
- net /MCU/INPUT_PIN renamed /MCU/PB4
- net /MCU/VOLT_SENSE renamed /MCU/PA1
- net /MCU/pU_COMP renamed /BEMF_Feedback/bU
- net /MCU/pV_COMP renamed /BEMF_Feedback/bV
- net /MCU/pW_COMP renamed /BEMF_Feedback/bW
- J2 pad 2: /PWM/SERVO_ISO -> /PWM/+5V_ISO
- J2 pad 3: /PWM/+5V_ISO -> /PWM/SERVO_ISO
- J3 pad 1: /CAN/GND_ISO1 -> /MCU/PA5
- U1 pad 1: /MCU/pU_HIGH -> /Gate_Drive/U_HIN
- U1 pad 2: /MCU/pU_LOW -> /Gate_Drive/U_LIN
- U2 pad 1: /MCU/pV_HIGH -> /Gate_Drive/V_HIN
- U2 pad 2: /MCU/pV_LOW -> /Gate_Drive/V_LIN
- U3 pad 1: /MCU/pW_HIGH -> /Gate_Drive/W_HIN
- U3 pad 2: /MCU/pW_LOW -> /Gate_Drive/W_LIN
Routing:
- net /CAN/CAN1_INT: track 39.2 -> 0.00 mm, vias 2 -> 0
- net /MCU/CURR_SENSE: track 39.1 -> 0.00 mm, vias 2 -> 0
- net /CAN/CAN1_INT_RX: track 38.8 -> 0.00 mm, vias 2 -> 0
- net /CAN/CAN1_INT_TX: track 36.3 -> 0.00 mm, vias 2 -> 0
- net +12V: track 61.1 -> 29.4 mm, vias 34 -> 32
- net Net-(IC1-Pad1): track 30.8 -> 0.00 mm, vias 2 -> 0
- net /CAN/CAN2_INT: track 29.6 -> 0.00 mm, vias 2 -> 0
- net Net-(IC1-Pad2): track 27.7 -> 0.00 mm, vias 2 -> 0
- net Net-(IC2-Pad2): track 25.5 -> 0.00 mm, vias 2 -> 0
- net /MCU/MOSI: track 22.5 -> 0.00 mm, vias 2 -> 0
- net /CAN/CAN2_INT_TX: track 21.4 -> 0.00 mm, vias 2 -> 0
- net Net-(IC2-Pad1): track 21.1 -> 0.00 mm, vias 2 -> 0
- net /Gate_Drive/U_HIN: track 0.00 -> 19.1 mm
- net /MCU/pU_HIGH: track 18.6 -> 0.00 mm
- net /MCU/MISO: track 18.6 -> 0.00 mm, vias 2 -> 0
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- added copper zone on In2.Cu, net GND
- removed copper zone on F.Cu, net +5V
- removed copper zone on In3.Cu, net +5V
Other:
- board size 50 x 67 mm -> 50 x 32 mm
- board text added: "I_SENSE"
- board text added: "Malloy Aeronautics STM32G071 Control Board V2.0"
- board text added: "S"
- board text removed: "STM32G071 CAN Control board V1.0"
