File: hw/ESC_Control_Board_STM32G071_V2.kicad_sch (KiCad schematic)
At the start: 5 parts, among them J2 Conn_01x03, J3 Conn_01x04, J4 Conn_01x04, J5 Conn_01x02, J6 Conn_01x15

Commit message: commenting
Parts:
- removed J3, J4: Conn_01x04, Connector_Molex:Molex_PicoBlade_53261-0471_1x04-1MP_P1.25mm_Horizontal, symbol Connector_Generic:Conn_01x04
- removed J5: Conn_01x02, Connector_Molex:Molex_PicoBlade_53261-0271_1x02-1MP_P1.25mm_Horizontal, symbol Connector_Generic:Conn_01x02
- added J3: Conn_01x01_Pin, TestPoint:TestPoint_Pad_1.0x1.0mm, symbol Connector:Conn_01x01_Pin
Connections:
- net MCU/PA5: now also J3.1 (Pin_1)
- net PWM/+5V_ISO: now also J2.2 (Pin_2); no longer J2.3 (Pin_3)
- net PWM/SERVO_ISO: now also J2.3 (Pin_3); no longer J2.2 (Pin_2)
Other:
- removed sheet CAN
- removed sheet Current_Sense
- sheet MCU ports: added PA1, PB1; removed PA0, PA4, PA6, PB10, PB11, PB12, PB15, PB5, PB6, PC0, PC1, PC2, PD6
- note added: "Current sense pad - Requires external shunt amplifier"
- note removed: "*To sense resistor 3x500uOhms"
- note removed: "CAN BUS 1"
- note removed: "CAN BUS 2"
- note removed: "Current sense resistor"
- moved on the sheet: J2, J6
