File: hw/PWM.kicad_sch (KiCad schematic)
At the start: 4 parts, among them IC5 ISO1540QDRQ1

Commit message: update comments
Parts:
- C24: Manufacturer_Name (none) -> Murata; Manufacturer_Part_Number (none) -> GRT188C81E475KE13D
Changed lines of the file:
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@@
+      (effects (font (size 1.27 1.27)) hide)
+    )
+    (property "Manufacturer_Name" "Murata" (id 4) (at 115.57 87.63 0)
+      (effects (font (size 1.27 1.27)) hide)
+    )
+    (property "Manufacturer_Part_Number" "GRT188C81E475KE13D " (id 5) (at 115.57 87.63 0)
       (effects (font (size 1.27 1.27)) hide)
     )
