File: hw/gate_drive.kicad_sch (KiCad schematic)
At the start: 30 parts, among them U1 L6498DTR, U2 L6498DTR, U3 L6498DTR, U4 ZXGD3006E6QTA, U5 ZXGD3006E6QTA, U6 ZXGD3006E6QTA, U7 ZXGD3006E6QTA, U8 ZXGD3006E6QTA, U9 ZXGD3006E6QTA

Commit message: update comments
Parts:
- C6, C7, C8: Manufacturer_Name (none) -> Murata; Manufacturer_Part_Number (none) -> GRT188C81E475KE13D
Changed lines of the file:
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@@
+      (effects (font (size 1.27 1.27)) hide)
+    )
+    (property "Manufacturer_Name" "Murata" (id 4) (at 121.92 138.43 0)
+      (effects (font (size 1.27 1.27)) hide)
+    )
+    (property "Manufacturer_Part_Number" "GRT188C81E475KE13D " (id 5) (at 121.92 138.43 0)
       (effects (font (size 1.27 1.27)) hide)
     )
@@
       (effects (font (size 1.27 1.27)) hide)
     )
+    (property "Manufacturer_Name" "Murata" (id 4) (at 121.92 40.64 0)
+      (effects (font (size 1.27 1.27)) hide)
+    )
+    (property "Manufacturer_Part_Number" "GRT188C81E475KE13D " (id 5) (at 121.92 40.64 0)
+      (effects (font (size 1.27 1.27)) hide)
+    )
     (pin "1")
     (pin "2")
@@
       (effects (font (size 1.27 1.27)) hide)
     )
+    (property "Manufacturer_Name" "Murata" (id 4) (at 121.92 88.9 0)
+      (effects (font (size 1.27 1.27)) hide)
+    )
+    (property "Manufacturer_Part_Number" "GRT188C81E475KE13D " (id 5) (at 121.92 88.9 0)
+      (effects (font (size 1.27 1.27)) hide)
+    )
